File: hyCyclePro_4ch.kicad_pcb (KiCad board)
At the start: 4 copper layers, 101.6 x 53.3 mm, 175 parts, among them J101 Conn_01x02, J102 Conn_01x01, J103 Conn_01x02, J104 Conn_01x01, J105 TWI0, J106 Conn_01x02, J107 Conn_01x01, J108 Conn_01x01, J109 Conn_01x01, J110 Conn_01x02, J111 Conn_01x01, J112 Conn_01x01, J113 Conn_01x01, J114 TWI1, J201 DUT, J301 DUT, J401 DUT, J501 DUT, P101 Power, P102 Analog, P103 GPIO, P104 Digital, P105 Serial, P106 Timer, P107 Serial, P108 CONN_01X01, P109 CONN_01X01, P110 CONN_01X01, P111 CONN_01X01, Q201 IRLML6244, Q202 IRLML6402, Q301 IRLML6244, Q302 IRLML6402, Q401 IRLML6244, Q402 IRLML6402, Q501 IRLML6244, Q502 IRLML6402, U101 MCP3564, U102 LM324, U103 LMV321, U104 MCP4728, U201 MAX4239AUT, U202 MAX4239AUT, U301 MAX4239AUT, U302 MAX4239AUT, U401 MAX4239AUT, U402 MAX4239AUT, U501 MAX4239AUT, U502 MAX4239AUT

Commit message: latest changes
Other:
- board text added: "this is an old version of the board with a few f*ckups."
Changed lines of the file:
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@@
-(kicad_pcb (version 20171130) (host pcbnew "(5.1.9)-1")
+(kicad_pcb (version 20171130) (host pcbnew 5.1.12-84ad8e8a86~92~ubuntu20.04.1)
   (general
     (thickness 1.6)
-    (drawings 10)
+    (drawings 11)
     (tracks 814)
     (zones 0)
@@
   (page A4)
   (title_block
-    (title hyCyclePro)
-    (date 2021-11-06)
-    (rev v1.0)
-    (company "Hyperstone GmbH")
-    (comment 1 4ch)
+    (title hyPrecessionCurrentMeasurment)
+    (date 2021-12-27)
+    (rev 0.1)
+    (company nerdyscout)
   )
   (layers
@@
     )
   )
+  (gr_text "this is an old version of the board with a few f*ckups." (at 154.559 61.976) (layer Cmts.User)
+    (effects (font (size 1.5 1.5) (thickness 0.3)))
+  )
   (gr_text hyCyclePro (at 171.704 95.631 90) (layer B.SilkS)
