File: hyCyclePro_4ch.sch (KiCad schematic (older format))
At the start: 44 parts, among them J101 Conn_01x02, J102 Conn_01x01, J103 Conn_01x02, J104 Conn_01x01, J105 TWI0, J106 Conn_01x02, J107 Conn_01x01, J110 Conn_01x02, J111 Conn_01x01, J114 TWI1, P101 Power, P102 Analog, P103 GPIO, P104 Digital, P105 Serial, P106 Timer, P107 Serial, P108 CONN_01X01, P109 CONN_01X01, P110 CONN_01X01, P111 CONN_01X01, U101 MCP3564, U103 LMV321

Commit message: latest changes
Parts:
- removed C112: 100n, Capacitor_SMD:C_0603_1608Metric, symbol Device:C
- removed JP105, JP106: Jumper_SolderJumper_2_Open, Jumper:SolderJumper-2_P1.3mm_Open_RoundedPad1.0x1.5mm, symbol Jumper:SolderJumper_2_Open
- removed R101: 270, Resistor_SMD:R_0603_1608Metric, symbol Device:R
- removed R106, R107: 100k 1%, Resistor_SMD:R_0603_1608Metric, symbol Device:R
- removed U103: LMV321, Package_TO_SOT_SMD:SOT-23-5, symbol Amplifier_Operational:LMV321
- added C? (x4): DNP, Capacitor_SMD:C_0402_1005Metric, symbol Device:C
Connections:
- net labels removed: VDD
- wire segments 185 -> 165
Other:
- note added: "TODO: connect to interrupt capable pin"
- note added: "TODO: connect to pin capable to generate 5MHz"
- note added: "external power source"
- note added: "internal"
- moved on the sheet: U101
