File: port.sch (KiCad schematic (older format))
At the start: 28 parts, among them J201 DUT, Q201 IRLML6244, Q202 IRLML6402, U201 MAX4239AUT, U202 MAX4239AUT

Commit message: latest changes
Parts:
- added C?: 100n, Capacitor_SMD:C_0603_1608Metric, symbol Device:C
- added R? (x2): 100k 1%, Resistor_SMD:R_0603_1608Metric, symbol Device:R
- added R?: 270, Resistor_SMD:R_0603_1608Metric, symbol Device:R
- added U?: LMV321, Package_TO_SOT_SMD:SOT-23-5, symbol Amplifier_Operational:LMV321
Connections:
- net GND: now also J201.1 (Pin_1); no longer C208.1, R203.1, R205.1, R208.1
- net GNDA: now also C?.1, R?.2, U?.2 (V-)
- net Power+: now also R203.2, R204.2; no longer J201.2 (Pin_2)
- net VDDA: now also C?.2, R?.1, U?.5 (V+)
- removed net Power-: J201.1 (Pin_1), R203.2, R204.2
- new net: R?.1, R?.2, U?.1 (+)
- new net: R?.2, U?.3 (-), U?.4
- new net ref: C208.1, J201.2 (Pin_2), R203.1, R205.1, R208.1, R?.1
Other:
- note added: "Here the device under test will be connected"
- note added: "Virtual GND"
- note added: "used to turn the DUT on/off"
- note removed: "Virtual GND with offset to analog GND"
- moved on the sheet: C301, C302, C303, C304, C305, C306, C307, C308, J301, Q301, Q302, R301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
